Commit message: add servingbot gazebo

File: serving_mobile/servingbot_description/urdf/servingbot.urdf (robot description, URDF)
Before this commit: robot servingbot, 4 links, 3 joints
Links:
- added link caster_back_link, mass 0.005; collision box size=0.040 0.010 0.040; visual box size=0.040 0.010 0.040
- added link caster_front_link, mass 0.005; collision box size=0.040 0.010 0.040; visual box size=0.040 0.010 0.040
Joints:
- added joint caster_back_joint: type fixed, parent base_link, child caster_back_link, origin xyz=-0.2885 0 -0.130 rpy=-1.57 0 0
- added joint caster_front_joint: type fixed, parent base_link, child caster_front_link, origin xyz=0.2885 0 -0.130 rpy=-1.57 0 0
- joint lidar_ref: origin xyz=0.24 0 0.08 rpy=3.14 0 -2.1329E-16 -> xyz=0.24 0 0.08 rpy=0 0 -2.1329E-16

File: serving_mobile/servingbot_description/urdf/servingbot.urdf (copy).xacro (robot description, xacro)
@@ -155,54 +155,4 @@
       </inertial>
   </link>
-  <joint name="caster_front_joint" type="fixed">
-    <parent link="base_link"/>
-    <child link="caster_front_link"/>
-    <origin xyz="0.2885 0 -0.210" rpy="-1.57 0 0"/>
-  </joint>
-  <link name="caster_front_link">
-    <!--visual>
-      <origin xyz="0 0.001 0" rpy="0 0 0"/>
-      <geometry>
-	<cylinder length="0.050" radius="0.05"/>
-      </geometry>
-    </visual-->
-    <collision>
-      <origin xyz="0 0.001 0" rpy="0 0 0"/>
-      <geometry>
-	<cylinder length="0.050" radius="0.05"/>
-        <!--box size="0.050 0.090 0.010"/-->
-      </geometry>
-    </collision>
-    <inertial>
-      <origin xyz="0 0 0"/>
-      <mass value="0.005"/>
-      <inertia ixx="0.001" ixy="0.0" ixz="0.0" iyy="0.001" iyz="0.0" izz="0.001"/>
-    </inertial>
-  </link>
-  <joint name="caster_back_joint" type="fixed">
-    <parent link="base_link"/>
-    <child link="caster_back_link"/>
-    <origin xyz="-0.2885 0 -0.210" rpy="-1.57 0 0"/>
-  </joint>
-  <link name="caster_back_link">
-    <!--visual>
-      <origin xyz="0 0.001 0" rpy="0 0 0"/>
-      <geometry>
-	<cylinder length="0.050" radius="0.05"/>
-      </geometry>
-    </visual-->
-    <collision>
-      <origin xyz="0 0.001 0" rpy="0 0 0"/>
-      <geometry>
-	<cylinder length="0.050" radius="0.05"/>
-        <!--box size="0.050 0.090 0.010"/-->
-      </geometry>
-    </collision>
-    <inertial>
-      <origin xyz="0 0 0"/>
-      <mass value="0.005"/>
-      <inertia ixx="0.001" ixy="0.0" ixz="0.0" iyy="0.001" iyz="0.0" izz="0.001"/>
-    </inertial>
-  </link>
   <joint
     name="lidar_joint"

File: serving_mobile/servingbot_description/urdf/servingbot_Gazebo.xacro (robot description, xacro)
@@ -56,14 +56,5 @@
     <material>Gazebo/FlatBlack</material>
   </gazebo>
-  <gazebo reference="caster_back_right_link">
-    <mu1>0.1</mu1>
-    <mu2>0.1</mu2>
-    <kp>1000000.0</kp>
-    <kd>100.0</kd>
-    <minDepth>0.001</minDepth>
-    <maxVel>1.0</maxVel>
-    <material>Gazebo/FlatBlack</material>
-  </gazebo>
-  <gazebo reference="caster_back_left_link">
+  <gazebo reference="caster_back_link">
     <mu1>0.1</mu1>
     <mu2>0.1</mu2>
