Commit message: add simulation

File: serving_mobile/servingbot_description/urdf/servingbot.urdf.xacro (robot description, xacro)
@@ -1,15 +1,39 @@
 <?xml version="1.0" ?>
 <robot name="servingbot" xmlns:xacro="http://ros.org/wiki/xacro">
-  <xacro:include filename="$(find zetabank_description)/urdf/common_properties.xacro"/>
-  <xacro:include filename="$(find zetabank_description)/urdf/zetabank.gazebo.xacro"/>
-  <link name="base_footprint"/>
-  <joint name="base_joint" type="fixed">
+  <xacro:include filename="$(find servingbot_description)/urdf/common_properties.xacro"/>
+  <xacro:include filename="$(find servingbot_description)/urdf/servingbot.gazebo.xacro"/>
+<!-- base -->
+<link name="base_footprint"/>
+ <joint name="base_joint" type="fixed">
     <parent link="base_footprint"/>
-    <child link="base_link"/>
-    <origin xyz="0.0 0.0 0.2465" rpy="0 0 0"/>
-  </joint>
-  <link name="body_link">
-    <visual>
-      <origin xyz="0 0 0" rpy="0 0 0"/>
+    <child link="base_link" />
+    <origin xyz="0 0 0.010" rpy="0 0 ${M_PI*0.5}"/>
+  </joint>
+  <link name="base_link">
+    <visual>
+      <origin xyz="-0 0 0.2465" rpy="0 0 ${-M_PI*0.5}"/>
+      <geometry>
+        <mesh filename="package://servingbot_description/meshes/body.STL"/>
+      </geometry>
+      <material name="light_black"/>
+    </visual>
+    <collision>
+      <origin xyz="0 0.064  0.048" rpy="0 0 ${M_PI*0.5}"/>
+      <geometry>
+        <box size="0.265 0.265 0.089"/>
+      </geometry>
+    </collision>
+    <inertial>
+      <origin xyz="0 0.064 0.048" rpy="0 0 ${M_PI*0.5}"/>
+      <mass value="0.01"/>
+      <inertia ixx="8.7002718e-03" ixy="-4.7576583e-05" ixz="1.1160499e-04"
+               iyy="8.6195418e-03" iyz="-3.5422299e-06"
+               izz="1.4612727e-02" />
+    </inertial>
+  </link>
+<!-- body -->
+ <link name="body_link">
+    <visual>
+      <origin xyz="-0 0 0.2465" rpy="0 0 ${-M_PI*0.5}"/>
       <geometry>
         <mesh filename="package://servingbot_description/meshes/base_plate.STL" />
@@ -21,18 +45,4 @@
       </material>
     </visual>
-    <collision>
-      <origin xyz="0 0 0" rpy="0 0 0"/>
-      <geometry>
-        <mesh
-          filename="package://servingbot_description/meshes/base_plate.STL" />
-      </geometry>
-    </collision>
-    <inertial>
-      <origin xyz="-0.0036904 0 0.0025" rpy="0 0 0"/>
-      <mass value="2"/>
-      <inertia ixx="0" ixy="0" ixz="0"
-               iyy="0" iyz="0"
-               izz="0" />
-    </inertial>
   </link>
   <joint
@@ -49,75 +59,35 @@
       xyz="0 0 0" />
   </joint>
-  <link
-    name="base_link">
-    <inertial>
-      <origin
-        xyz="-0.0070361 -0.0010307 -0.094165"
-        rpy="0 0 0" />
-      <mass
-        value="7" />
-      <inertia
-        ixx="0.114"
-        ixy="3.4187E-05"
-        ixz="-0.0079587"
-        iyy="0.084746"
-        iyz="-0.00069939"
-        izz="0.14914" />
-    </inertial>
-    <visual>
-      <origin
-        xyz="0 0 0"
-        rpy="0 0 0" />
-      <geometry>
-        <mesh
-          filename="package://servingbot_description/meshes/body.STL" />
-      </geometry>
-      <material
-        name="">
-        <color
-          rgba="0.79216 0.81961 0.93333 1" />
-      </material>
-    </visual>
-    <collision>
-      <origin
-        xyz="0 0 0"
-        rpy="0 0 0" />
-      <geometry>
-        <mesh
-          filename="package://servingbot_description/meshes/body.STL" />
-      </geometry>
-    </collision>
-  </link>
-  <joint name="wheel_left_joint" type="continuous">
+<!-- wheel -->
+<joint name="wheel_left_joint" type="continuous">
     <parent link="base_link"/>
     <child link="wheel_left_link"/>
-    <origin xyz="-0.0010943 0.28875 -0.145" rpy="-2.2643E-16 1.1179E-16 2.2128E-16"/>
-    <axis xyz="0 1 0"/>
+    <origin xyz="0.280 0.0  0.100" rpy="${-M_PI*0.5} 0 ${-M_PI*0.5}"/>
+    <axis xyz="0 0 1"/>
   </joint>
   <link name="wheel_left_link">
-    <visual>
-      <origin xyz="0 0 0" rpy="0 0 0"/>
-      <geometry>
-        <mesh filename="package://servingbot_description/meshes/left_wheel.STL" />
-      </geometry>
-      <material
-        name="">
-        <color
-          rgba="0.79216 0.81961 0.93333 1" />
-      </material>
-    </visual>
-    <collision>
-      <origin xyz="0 0 0" rpy="0 0 0"/>
-      <geometry>
-        <mesh
-          filename="package://servingbot_description/meshes/left_wheel.STL" />
-      </geometry>
-    </collision>
-    <inertial>
-      <origin xyz="0 0 0" />
-      <mass value="3.5" />
-      <inertia ixx="0" ixy="0" ixz="0"
-               iyy="0" iyz="0"
-               izz="0" />
+     <visual>
+      <origin xyz="0 0 0" rpy="${-M_PI*0.5} 0 0"/>
+      <geometry>
+        <mesh filename="package://servingbot_description/meshes/left_wheel.STL"/>
+      </geometry>
+      <material
+        name="">
+        <color
+          rgba="0.79216 0.81961 0.93333 1" />
+      </material>
+    </visual>
+    <collision>
+      <origin rpy="0 0 0" xyz="0 0 0"/>
+      <geometry>
+        <cylinder length="0.050" radius="0.100"/>
+      </geometry>
+    </collision>
+    <inertial>
+      <origin xyz="0 0 0" />
+      <mass value="2.8498940e-02" />
+      <inertia ixx="1.1175580e-05" ixy="-4.2369783e-11" ixz="-5.9381719e-09"
+               iyy="1.1192413e-05" iyz="-1.4400107e-11"
+               izz="2.0712558e-05" />
       </inertial>
   </link>
@@ -125,10 +95,10 @@
     <parent link="base_link"/>
     <child link="wheel_right_link"/>
-    <origin xyz="-0.0010943 -0.2675 -0.145" rpy="-5.2266E-18 -5.5914E-16 8.922E-16"/>
-    <axis xyz="0 1 0"/>
+    <origin xyz="-0.280 0.0  0.100" rpy="${-M_PI*0.5} 0 ${-M_PI*0.5}"/>
+    <axis xyz="0 0 1"/>
   </joint>
   <link name="wheel_right_link">
     <visual>
-      <origin xyz="0 0 0" rpy="0 0 0"/>
+      <origin xyz="0 0 -0.025" rpy="${-M_PI*0.5} 0 0"/>
       <geometry>
         <mesh filename="package://servingbot_description/meshes/right_wheel.STL"/>
@@ -141,81 +111,79 @@
     </visual>
     <collision>
-      <origin xyz="0 0 0" rpy="0 0 0"/>
-      <geometry>
-        <mesh
-          filename="package://servingbot_description/meshes/right_wheel.STL" />
-      </geometry>
-    </collision>
-    <inertial>
-      <origin xyz="0 -5.5511E-17 0" />
-      <mass value="3.5" />
-      <inertia ixx="0" ixy="0" ixz="0"
-               iyy="0" iyz="0"
-               izz="0" />
+      <origin rpy="0 0 0" xyz="0 0 0"/>
+      <geometry>
+        <cylinder length="0.050" radius="0.100"/>
+      </geometry>
+    </collision>
+    <inertial>
+      <origin xyz="0 0 0" />
+      <mass value="2.8498940e-02" />
+      <inertia ixx="1.1175580e-05" ixy="-4.2369783e-11" ixz="-5.9381719e-09"
+               iyy="1.1192413e-05" iyz="-1.4400107e-11"
+               izz="2.0712558e-05" />
       </inertial>
   </link>
+<!-- caster -->
+  <joint name="caster_back_left_joint" type="fixed">
+    <parent link="base_link"/>
+    <child link="caster_back_left_link"/>
+    <origin xyz="-0.177 0.264 0.008" rpy="${-M_PI*0.5} 0 ${-M_PI*0.5}"/>
+  </joint>
+  <link name="caster_back_left_link">
+    <collision>
+      <origin xyz="0 0.001 0" rpy="0 0 0"/>
+      <geometry>
+        <box size="0.030 0.009 0.020"/>
+      </geometry>
+    </collision>
+    <inertial>
+      <origin xyz="0 0 0" />
+      <mass value="0.005" />
+      <inertia ixx="0.001" ixy="0.0" ixz="0.0"
+               iyy="0.001" iyz="0.0"
+               izz="0.001" />
+    </inertial>
+  </link>
+  <joint name="caster_back_right_joint" type="fixed">
+    <parent link="base_link"/>
+    <child link="caster_back_right_link"/>
+    <origin xyz="0.177 0.264 0.008" rpy="${-M_PI*0.5} 0 ${-M_PI*0.5}"/>
+  </joint>
+  <link name="caster_back_right_link">
+    <collision>
+      <origin xyz="0 0.001 0" rpy="0 0 0"/>
+      <geometry>
+        <box size="0.030 0.009 0.020"/>
+      </geometry>
+    </collision>
+    <inertial>
+      <origin xyz="0 0 0" />
+      <mass value="0.005" />
+      <inertia ixx="0.001" ixy="0.0" ixz="0.0"
+               iyy="0.001" iyz="0.0"
+               izz="0.001" />
+    </inertial>
+  </link>
   <joint name="caster_front_joint" type="fixed">
     <parent link="base_link"/>
     <child link="caster_front_link"/>
-    <origin xyz="0.2885 0 -0.210" rpy="-1.57 0 0"/>
+    <origin xyz="0 -0.150 0.020" rpy="${-M_PI*0.5} 0 ${-M_PI*0.5}"/>
   </joint>
   <link name="caster_front_link">
-    <!--visual>
+    <collision>
       <origin xyz="0 0.001 0" rpy="0 0 0"/>
       <geometry>
-	<cylinder length="0.050" radius="0.05"/>
-      </geometry>
-    </visual-->
-    <collision>
-      <origin xyz="0 0.001 0" rpy="0 0 0"/>
-      <geometry>
-	<cylinder length="0.050" radius="0.05"/>
-        <!--box size="0.050 0.090 0.010"/-->
-      </geometry>
-    </collision>
-    <inertial>
-      <origin xyz="0 0 0"/>
-      <mass value="0.005"/>
-      <inertia ixx="0.001" ixy="0.0" ixz="0.0" iyy="0.001" iyz="0.0" izz="0.001"/>
-    </inertial>
-  </link>
-  <joint name="caster_back_joint" type="fixed">
-    <parent link="base_link"/>
-    <child link="caster_back_link"/>
-    <origin xyz="-0.2885 0 -0.210" rpy="-1.57 0 0"/>
-  </joint>
-  <link name="caster_back_link">
-    <!--visual>
-      <origin xyz="0 0.001 0" rpy="0 0 0"/>
-      <geometry>
-	<cylinder length="0.050" radius="0.05"/>
-      </geometry>
-    </visual-->
-    <collision>
-      <origin xyz="0 0.001 0" rpy="0 0 0"/>
-      <geometry>
-	<cylinder length="0.050" radius="0.05"/>
-        <!--box size="0.050 0.090 0.010"/-->
-      </geometry>
-    </collision>
-    <inertial>
-      <origin xyz="0 0 0"/>
-      <mass value="0.005"/>
-      <inertia ixx="0.001" ixy="0.0" ixz="0.0" iyy="0.001" iyz="0.0" izz="0.001"/>
-    </inertial>
-  </link>
-  <joint
-    name="lidar_joint"
-    type="fixed">
-    <origin
-      xyz="0.23721 0 0.0453"
-      rpy="0 1.111E-15 0" />
-    <parent
-      link="base_link" />
-    <child
-      link="lidar_link" />
-    <axis
-      xyz="0 0 0" />
-  </joint>
+        <box size="0.030 0.009 0.020"/>
+      </geometry>
+    </collision>
+    <inertial>
+      <origin xyz="0 0 0" />
+      <mass value="0.005" />
+      <inertia ixx="0.001" ixy="0.0" ixz="0.0"
+               iyy="0.001" iyz="0.0"
+               izz="0.001" />
+    </inertial>
+  </link>
+<!-- imu -->
   <joint name="imu_joint" type="fixed">
     <parent link="base_link"/>
@@ -224,43 +192,22 @@
   </joint>
   <link name="imu_link"/>
-  <link
-    name="lidar_link">
-    <inertial>
-      <origin
-        xyz="-0.25974 -0.001068 -0.098004"
-        rpy="0 0 3.141592" />
-      <mass
-        value="0.05" />
-      <inertia
-        ixx="6.003E-06"
-        ixy="2.5645E-07"
-        ixz="-2.0674E-06"
-        iyy="8.525E-06"
-        iyz="7.9724E-08"
-        izz="3.7518E-06" />
-    </inertial>
-    <visual>
-      <origin
-        xyz="0 0 0"
-        rpy="0 0 3.141592" />
-      <geometry>
-        <mesh
-          filename="package://servingbot_description/meshes/lidar.STL" />
-      </geometry>
-      <material
-        name="">
-        <color
-          rgba="0.79216 0.81961 0.93333 1" />
-      </material>
-    </visual>
-    <collision>
-      <origin
-        xyz="0 0 0"
-        rpy="0 0 0" />
-      <geometry>
-        <mesh
-          filename="package://servingbot_description/meshes/lidar.STL" />
-      </geometry>
-    </collision>
+<!-- scan -->
+  <joint name="lidar_joint" type="fixed">
+    <parent link="base_link"/>
+    <child link="lidar_link"/>
+    <origin xyz="0 -0.28 0.21" rpy="0 0 ${-M_PI*0.5}"/>
+  </joint>
+  <link name="lidar_link">
+    <visual>
+      <origin xyz="0 0 0" rpy="0 0 0"/>
+      <geometry>
+        <mesh filename="package://servingbot_description/meshes/lidar.STL" />
+      </geometry>
+      <material
+        name="">
+        <color
+          rgba="0.79216 0.81961 0.93333 1" />
+      </material>
+    </visual>
   </link>
 </robot>

File: serving_mobile/servingbot_description/urdf/servingbot3.gazebo.xacro (robot description, xacro)
@@ -17,7 +17,7 @@
       <leftJoint>wheel_left_joint</leftJoint>
       <rightJoint>wheel_right_joint</rightJoint>
-      <wheelSeparation>0.36</wheelSeparation>
+      <wheelSeparation>0.58</wheelSeparation>
       <!-- >wheelDiameter>0.0812</wheelDiameter-->
-      <wheelDiameter>0.1624</wheelDiameter>
+      <wheelDiameter>0.200</wheelDiameter>
       <wheelAcceleration>1</wheelAcceleration>
       <wheelTorque>100</wheelTorque>
