Commit message: add gpu_ray

File: serving_mobile/servingbot_description/urdf/rl_servingbot.gazebo.xacro (robot description, xacro)
@@ -1,3 +1,2 @@
-<<<<<<< HEAD
 <?xml version="1.0"?>
 <robot name="servingbot_sim" xmlns:xacro="http://ros.org/wiki/xacro">
@@ -143,148 +142,3 @@
     </sensor>
   </gazebo>
-=======
-<?xml version="1.0"?>
-<robot name="servingbot_sim" xmlns:xacro="http://ros.org/wiki/xacro">
-  <xacro:arg name="laser_visual" default="false"/>
-  <xacro:arg name="imu_visual"   default="false"/>
-  <xacro:arg name="imu_visual"    default="false"/>
-  <xacro:arg name="lidar_visual"    default="true"/>
-  <gazebo reference="base_link">
-    <material>Gazebo/DarkGrey</material>
-  </gazebo>
-  <gazebo reference="wheel_left_link">
-    <mu1>10</mu1>
-    <mu2>10</mu2>
-    <kp>100000.0</kp>
-    <kd>10.0</kd>
-    <minDepth>0.001</minDepth>
-    <maxVel>2.0</maxVel>
-    <fdir1>1 0 0</fdir1>
-    <material>Gazebo/FlatBlack</material>
-  </gazebo>
-  <gazebo reference="wheel_right_link">
-    <mu1>10</mu1>
-    <mu2>10</mu2>
-    <kp>100000.0</kp>
-    <kd>10.0</kd>
-    <minDepth>0.001</minDepth>
-    <maxVel>2.0</maxVel>
-    <fdir1>1 0 0</fdir1>
-    <material>Gazebo/FlatBlack</material>
-  </gazebo>
-  <gazebo reference="caster_front_link">
-    <mu1>0.1</mu1>
-    <mu2>0.1</mu2>
-    <kp>1000000.0</kp>
-    <kd>100.0</kd>
-    <minDepth>0.001</minDepth>
-    <maxVel>1.0</maxVel>
-    <material>Gazebo/FlatBlack</material>
-  </gazebo>
-    <gazebo reference="caster_back_left_link">
-    <mu1>0.1</mu1>
-    <mu2>0.1</mu2>
-    <kp>1000000.0</kp>
-    <kd>100.0</kd>
-    <minDepth>0.001</minDepth>
-    <maxVel>1.0</maxVel>
-    <material>Gazebo/FlatBlack</material>
-  </gazebo>
-  <gazebo reference="caster_back_right_link">
-    <mu1>0.1</mu1>
-    <mu2>0.1</mu2>
-    <kp>1000000.0</kp>
-    <kd>100.0</kd>
-    <minDepth>0.001</minDepth>
-    <maxVel>1.0</maxVel>
-    <material>Gazebo/FlatBlack</material>
-  </gazebo>
-  <gazebo reference="imu_link">
-    <sensor type="imu" name="imu">
-      <always_on>true</always_on>
-      <update_rate>50</update_rate>
-      <visualize>$(arg imu_visual)</visualize>
-    </sensor>
-    <material>Gazebo/FlatBlack</material>
-  </gazebo>
-  <gazebo>
-    <plugin name="servingbot_controller" filename="libgazebo_ros_diff_drive.so">
-      <commandTopic>cmd_vel</commandTopic>
-      <odometryTopic>odom</odometryTopic>
-      <odometryFrame>odom</odometryFrame>
-      <odometrySource>world</odometrySource>
-      <publishOdomTF>true</publishOdomTF>
-      <robotBaseFrame>base_footprint</robotBaseFrame>
-      <publishWheelTF>false</publishWheelTF>
-      <publishWheelJointState>true</publishWheelJointState>
-      <legacyMode>false</legacyMode>
-      <updateRate>10</updateRate>
-      <leftJoint>wheel_left_joint</leftJoint>
-      <rightJoint>wheel_right_joint</rightJoint>
-      <wheelSeparation>0.56</wheelSeparation>
-      <wheelDiameter>0.200</wheelDiameter>
-      <wheelAcceleration>1</wheelAcceleration>
-      <wheelTorque>100</wheelTorque>
-    </plugin>
-  </gazebo>
-  <gazebo>
-    <plugin name="imu_plugin" filename="libgazebo_ros_imu.so">
-      <alwaysOn>true</alwaysOn>
-      <bodyName>imu_link</bodyName>
-      <topicName>/imu</topicName>
-      <serviceName>/imu_service</serviceName>
-      <gaussianNoise>0.0</gaussianNoise>
-      <updateRate>100.0</updateRate>
-      <imu>
-        <noise>
-          <type>gaussian</type>
-          <rate>
-            <mean>0.0</mean>
-            <stddev>2e-4</stddev>
-            <bias_mean>0.0000075</bias_mean>
-            <bias_stddev>0.0000008</bias_stddev>
-          </rate>
-          <accel>
-            <mean>0.0</mean>
-            <stddev>1.7e-2</stddev>
-            <bias_mean>0.1</bias_mean>
-            <bias_stddev>0.001</bias_stddev>
-          </accel>
-        </noise>
-      </imu>
-    </plugin>
-  </gazebo>
-  <gazebo reference="lidar_link">
-    <material>Gazebo/FlatBlack</material>
-    <sensor type="ray" name="lds_lfcd_sensor">
-      <pose>0 0 0 0 0 1.57079631</pose>
-      <visualize>$(arg lidar_visual)</visualize>
-      <update_rate>512</update_rate>
-      <ray>
-        <scan>
-          <horizontal>
-            <samples>270</samples>
-            <resolution>1</resolution>
-            <min_angle>-2.1</min_angle>
-            <max_angle>2.1</max_angle>
-          </horizontal>
-        </scan>
-        <range>
-          <min>0.05</min>
-          <max>6.0</max>
-          <resolution>0.009</resolution>
-        </range>
-        <noise>
-          <type>gaussian</type>
-          <mean>0.0</mean>
-          <stddev>0.01</stddev>
-        </noise>
-      </ray>
-      <plugin name="gazebo_ros_lds_lfcd_controller" filename="libgazebo_ros_laser.so">
-        <topicName>/scan</topicName>
-        <frameName>lidar_link</frameName>
-      </plugin>
-    </sensor>
-  </gazebo>
->>>>>>> 80fafc819a0753ed1204de4e163596fdf3e497fe
 </robot>

File: serving_mobile/servingbot_description/urdf/servingbot_rl.gazebo.xacro (robot description, xacro)
@@ -1,3 +1,2 @@
-<<<<<<< HEAD
 <?xml version="1.0"?>
 <robot name="servingbot_sim" xmlns:xacro="http://ros.org/wiki/xacro">
@@ -115,5 +114,5 @@
     <sensor type="gpu_ray" name="lds_lfcd_sensor">
       <pose>0 0 0 0 0 1.57079631</pose>
-      <visualize>$(arg lidar_visual)</visualize>
+      <visualize>true</visualize>
       <update_rate>1500</update_rate>
       <ray>
@@ -137,5 +136,5 @@
         </noise>
       </ray>
-      <plugin name="gazebo_ros_lds_lfcd_controller" filename="libgazebo_ros_gpu_laser.so">
+      <plugin name="gazebo_ros_lds_lfcd_controller" filename="libgazebo_gpu_ros_laser.so">
         <topicName>/scan</topicName>
         <frameName>lidar_link</frameName>
@@ -143,148 +142,3 @@
     </sensor>
   </gazebo>
-=======
-<?xml version="1.0"?>
-<robot name="servingbot_sim" xmlns:xacro="http://ros.org/wiki/xacro">
-  <xacro:arg name="laser_visual" default="false"/>
-  <xacro:arg name="imu_visual"   default="false"/>
-  <xacro:arg name="imu_visual"    default="false"/>
-  <xacro:arg name="lidar_visual"    default="true"/>
-  <gazebo reference="base_link">
-    <material>Gazebo/DarkGrey</material>
-  </gazebo>
-  <gazebo reference="wheel_left_link">
-    <mu1>10</mu1>
-    <mu2>10</mu2>
-    <kp>100000.0</kp>
-    <kd>10.0</kd>
-    <minDepth>0.001</minDepth>
-    <maxVel>2.0</maxVel>
-    <fdir1>1 0 0</fdir1>
-    <material>Gazebo/FlatBlack</material>
-  </gazebo>
-  <gazebo reference="wheel_right_link">
-    <mu1>10</mu1>
-    <mu2>10</mu2>
-    <kp>100000.0</kp>
-    <kd>10.0</kd>
-    <minDepth>0.001</minDepth>
-    <maxVel>2.0</maxVel>
-    <fdir1>1 0 0</fdir1>
-    <material>Gazebo/FlatBlack</material>
-  </gazebo>
-  <gazebo reference="caster_front_link">
-    <mu1>0.1</mu1>
-    <mu2>0.1</mu2>
-    <kp>1000000.0</kp>
-    <kd>100.0</kd>
-    <minDepth>0.001</minDepth>
-    <maxVel>1.0</maxVel>
-    <material>Gazebo/FlatBlack</material>
-  </gazebo>
-    <gazebo reference="caster_back_left_link">
-    <mu1>0.1</mu1>
-    <mu2>0.1</mu2>
-    <kp>1000000.0</kp>
-    <kd>100.0</kd>
-    <minDepth>0.001</minDepth>
-    <maxVel>1.0</maxVel>
-    <material>Gazebo/FlatBlack</material>
-  </gazebo>
-  <gazebo reference="caster_back_right_link">
-    <mu1>0.1</mu1>
-    <mu2>0.1</mu2>
-    <kp>1000000.0</kp>
-    <kd>100.0</kd>
-    <minDepth>0.001</minDepth>
-    <maxVel>1.0</maxVel>
-    <material>Gazebo/FlatBlack</material>
-  </gazebo>
-  <gazebo reference="imu_link">
-    <sensor type="imu" name="imu">
-      <always_on>true</always_on>
-      <update_rate>50</update_rate>
-      <visualize>$(arg imu_visual)</visualize>
-    </sensor>
-    <material>Gazebo/FlatBlack</material>
-  </gazebo>
-  <gazebo>
-    <plugin name="servingbot_controller" filename="libgazebo_ros_diff_drive.so">
-      <commandTopic>cmd_vel</commandTopic>
-      <odometryTopic>odom</odometryTopic>
-      <odometryFrame>odom</odometryFrame>
-      <odometrySource>world</odometrySource>
-      <publishOdomTF>true</publishOdomTF>
-      <robotBaseFrame>base_footprint</robotBaseFrame>
-      <publishWheelTF>false</publishWheelTF>
-      <publishWheelJointState>true</publishWheelJointState>
-      <legacyMode>false</legacyMode>
-      <updateRate>10</updateRate>
-      <leftJoint>wheel_left_joint</leftJoint>
-      <rightJoint>wheel_right_joint</rightJoint>
-      <wheelSeparation>0.56</wheelSeparation>
-      <wheelDiameter>0.200</wheelDiameter>
-      <wheelAcceleration>1</wheelAcceleration>
-      <wheelTorque>100</wheelTorque>
-    </plugin>
-  </gazebo>
-  <gazebo>
-    <plugin name="imu_plugin" filename="libgazebo_ros_imu.so">
-      <alwaysOn>true</alwaysOn>
-      <bodyName>imu_link</bodyName>
-      <topicName>/imu</topicName>
-      <serviceName>/imu_service</serviceName>
-      <gaussianNoise>0.0</gaussianNoise>
-      <updateRate>100.0</updateRate>
-      <imu>
-        <noise>
-          <type>gaussian</type>
-          <rate>
-            <mean>0.0</mean>
-            <stddev>2e-4</stddev>
-            <bias_mean>0.0000075</bias_mean>
-            <bias_stddev>0.0000008</bias_stddev>
-          </rate>
-          <accel>
-            <mean>0.0</mean>
-            <stddev>1.7e-2</stddev>
-            <bias_mean>0.1</bias_mean>
-            <bias_stddev>0.001</bias_stddev>
-          </accel>
-        </noise>
-      </imu>
-    </plugin>
-  </gazebo>
-  <gazebo reference="lidar_link">
-    <material>Gazebo/FlatBlack</material>
-    <sensor type="ray" name="lds_lfcd_sensor">
-      <pose>0 0 0 0 0 1.57079631</pose>
-      <visualize>$(arg lidar_visual)</visualize>
-      <update_rate>512</update_rate>
-      <ray>
-        <scan>
-          <horizontal>
-            <samples>270</samples>
-            <resolution>1</resolution>
-            <min_angle>-2.1</min_angle>
-            <max_angle>2.1</max_angle>
-          </horizontal>
-        </scan>
-        <range>
-          <min>0.05</min>
-          <max>6.0</max>
-          <resolution>0.009</resolution>
-        </range>
-        <noise>
-          <type>gaussian</type>
-          <mean>0.0</mean>
-          <stddev>0.01</stddev>
-        </noise>
-      </ray>
-      <plugin name="gazebo_ros_lds_lfcd_controller" filename="libgazebo_ros_laser.so">
-        <topicName>/scan</topicName>
-        <frameName>lidar_link</frameName>
-      </plugin>
-    </sensor>
-  </gazebo>
->>>>>>> 80fafc819a0753ed1204de4e163596fdf3e497fe
 </robot>

File: serving_mobile/servingbot_description/urdf/servingbot_rl.urdf.xacro (robot description, xacro)
@@ -1,3 +1,2 @@
-<<<<<<< HEAD
 <?xml version="1.0" ?>
 <robot name="servingbot" xmlns:xacro="http://ros.org/wiki/xacro">
@@ -212,217 +211,3 @@
     </visual>
   </link>
-=======
-<?xml version="1.0" ?>
-<robot name="servingbot" xmlns:xacro="http://ros.org/wiki/xacro">
-  <xacro:include filename="$(find servingbot_description)/urdf/common_properties.xacro"/>
-  <xacro:include filename="$(find servingbot_description)/urdf/servingbot_rl.gazebo.xacro"/>
-<!-- base -->
-<link name="base_footprint"/>
- <joint name="base_joint" type="fixed">
-    <parent link="base_footprint"/>
-    <child link="base_link" />
-    <origin xyz="0 0 0.010" rpy="0 0 ${M_PI*0.5}"/>
-  </joint>
-  <link name="base_link">
-    <visual>
-      <origin xyz="-0 0 0.2465" rpy="0 0 ${-M_PI*0.5}"/>
-      <geometry>
-        <mesh filename="package://servingbot_description/meshes/body.STL"/>
-      </geometry>
-      <material name="light_black"/>
-    </visual>
-    <collision>
-      <origin xyz="0 0.064  0.048" rpy="0 0 ${M_PI*0.5}"/>
-      <geometry>
-        <box size="0.265 0.265 0.089"/>
-      </geometry>
-    </collision>
-    <inertial>
-      <origin xyz="0 0.064 0.048" rpy="0 0 ${M_PI*0.5}"/>
-      <mass value="0.01"/>
-      <inertia ixx="8.7002718e-03" ixy="-4.7576583e-05" ixz="1.1160499e-04"
-               iyy="8.6195418e-03" iyz="-3.5422299e-06"
-               izz="1.4612727e-02" />
-    </inertial>
-  </link>
-<!-- body -->
- <link name="body_link">
-    <visual>
-      <origin xyz="-0 0 0.2465" rpy="0 0 ${-M_PI*0.5}"/>
-      <geometry>
-        <mesh filename="package://servingbot_description/meshes/base_plate.STL" />
-      </geometry>
-      <material
-        name="">
-        <color
-          rgba="0.79216 0.81961 0.93333 1" />
-      </material>
-    </visual>
-  </link>
-  <joint
-    name="body_joint"
-    type="fixed">
-    <origin
-      xyz="0.0039057 0 -0.08"
-      rpy="-6.913E-15 -1.1102E-16 -5.4234E-31" />
-    <parent
-      link="base_link" />
-    <child
-      link="body_link" />
-    <axis
-      xyz="0 0 0" />
-  </joint>
-<!-- wheel -->
-<joint name="wheel_left_joint" type="continuous">
-    <parent link="base_link"/>
-    <child link="wheel_left_link"/>
-    <origin xyz="0.280 0.0  0.100" rpy="${-M_PI*0.5} 0 ${-M_PI*0.5}"/>
-    <axis xyz="0 0 1"/>
-  </joint>
-  <link name="wheel_left_link">
-     <visual>
-      <origin xyz="0 0 0" rpy="${-M_PI*0.5} 0 0"/>
-      <geometry>
-        <mesh filename="package://servingbot_description/meshes/left_wheel.STL"/>
-      </geometry>
-      <material
-        name="">
-        <color
-          rgba="0.79216 0.81961 0.93333 1" />
-      </material>
-    </visual>
-    <collision>
-      <origin rpy="0 0 0" xyz="0 0 0"/>
-      <geometry>
-        <cylinder length="0.050" radius="0.100"/>
-      </geometry>
-    </collision>
-    <inertial>
-      <origin xyz="0 0 0" />
-      <mass value="2.8498940e-02" />
-      <inertia ixx="1.1175580e-05" ixy="-4.2369783e-11" ixz="-5.9381719e-09"
-               iyy="1.1192413e-05" iyz="-1.4400107e-11"
-               izz="2.0712558e-05" />
-      </inertial>
-  </link>
-  <joint name="wheel_right_joint" type="continuous">
-    <parent link="base_link"/>
-    <child link="wheel_right_link"/>
-    <origin xyz="-0.280 0.0  0.100" rpy="${-M_PI*0.5} 0 ${-M_PI*0.5}"/>
-    <axis xyz="0 0 1"/>
-  </joint>
-  <link name="wheel_right_link">
-    <visual>
-      <origin xyz="0 0 -0.025" rpy="${-M_PI*0.5} 0 0"/>
-      <geometry>
-        <mesh filename="package://servingbot_description/meshes/right_wheel.STL"/>
-      </geometry>
-      <material
-        name="">
-        <color
-          rgba="0.79216 0.81961 0.93333 1" />
-      </material>
-    </visual>
-    <collision>
-      <origin rpy="0 0 0" xyz="0 0 0"/>
-      <geometry>
-        <cylinder length="0.050" radius="0.100"/>
-      </geometry>
-    </collision>
-    <inertial>
-      <origin xyz="0 0 0" />
-      <mass value="2.8498940e-02" />
-      <inertia ixx="1.1175580e-05" ixy="-4.2369783e-11" ixz="-5.9381719e-09"
-               iyy="1.1192413e-05" iyz="-1.4400107e-11"
-               izz="2.0712558e-05" />
-      </inertial>
-  </link>
-<!-- caster -->
-  <joint name="caster_back_left_joint" type="fixed">
-    <parent link="base_link"/>
-    <child link="caster_back_left_link"/>
-    <origin xyz="-0.177 0.264 0.008" rpy="${-M_PI*0.5} 0 ${-M_PI*0.5}"/>
-  </joint>
-  <link name="caster_back_left_link">
-    <collision>
-      <origin xyz="0 0.001 0" rpy="0 0 0"/>
-      <geometry>
-        <box size="0.030 0.009 0.020"/>
-      </geometry>
-    </collision>
-    <inertial>
-      <origin xyz="0 0 0" />
-      <mass value="0.005" />
-      <inertia ixx="0.001" ixy="0.0" ixz="0.0"
-               iyy="0.001" iyz="0.0"
-               izz="0.001" />
-    </inertial>
-  </link>
-  <joint name="caster_back_right_joint" type="fixed">
-    <parent link="base_link"/>
-    <child link="caster_back_right_link"/>
-    <origin xyz="0.177 0.264 0.008" rpy="${-M_PI*0.5} 0 ${-M_PI*0.5}"/>
-  </joint>
-  <link name="caster_back_right_link">
-    <collision>
-      <origin xyz="0 0.001 0" rpy="0 0 0"/>
-      <geometry>
-        <box size="0.030 0.009 0.020"/>
-      </geometry>
-    </collision>
-    <inertial>
-      <origin xyz="0 0 0" />
-      <mass value="0.005" />
-      <inertia ixx="0.001" ixy="0.0" ixz="0.0"
-               iyy="0.001" iyz="0.0"
-               izz="0.001" />
-    </inertial>
-  </link>
-  <joint name="caster_front_joint" type="fixed">
-    <parent link="base_link"/>
-    <child link="caster_front_link"/>
-    <origin xyz="0 -0.150 0.020" rpy="${-M_PI*0.5} 0 ${-M_PI*0.5}"/>
-  </joint>
-  <link name="caster_front_link">
-    <collision>
-      <origin xyz="0 0.001 0" rpy="0 0 0"/>
-      <geometry>
-        <box size="0.030 0.009 0.020"/>
-      </geometry>
-    </collision>
-    <inertial>
-      <origin xyz="0 0 0" />
-      <mass value="0.005" />
-      <inertia ixx="0.001" ixy="0.0" ixz="0.0"
-               iyy="0.001" iyz="0.0"
-               izz="0.001" />
-    </inertial>
-  </link>
-<!-- imu -->
-  <joint name="imu_joint" type="fixed">
-    <parent link="base_link"/>
-    <child link="imu_link"/>
-    <origin xyz="0.0 -0.07 0.37" rpy="0 0 ${-M_PI*0.5}"/>
-  </joint>
-  <link name="imu_link"/>
-<!-- scan -->
-  <joint name="lidar_joint" type="fixed">
-    <parent link="base_link"/>
-    <child link="lidar_link"/>
-    <origin xyz="0 -0.28 0.21" rpy="0 0 ${-M_PI*0.5}"/>
-  </joint>
-  <link name="lidar_link">
-    <visual>
-      <origin xyz="0 0 0" rpy="0 0 0"/>
-      <geometry>
-        <mesh filename="package://servingbot_description/meshes/lidar.STL" />
-      </geometry>
-      <material
-        name="">
-        <color
-          rgba="0.79216 0.81961 0.93333 1" />
-      </material>
-    </visual>
-  </link>
->>>>>>> 80fafc819a0753ed1204de4e163596fdf3e497fe
 </robot>
